File: FlexLogicMini_EVB.kicad_pcb (KiCad board)
At the start: 8 copper layers, 50 x 50 mm, 209 parts, among them IC1 MT9700, IC2 SL2.1s, IC3 W25Q16JVUXIQ, IC4 LCMXO2-1200HC-4SG32I, IC5 MTS4P, J1 GT-USB-7010ASV, J10 Conn_01x04, J11 Conn_02x03_Odd_Even, J12 1.0-3PWB, J13 PH-2A, J2 WJ126V-5.0-2P, J3 WJ126V-5.0-2P, J4 WJ126V-5.0-2P, J5 WJ126V-5.0-2P, J6 Conn_02x03_Odd_Even, J7 Conn_02x03_Odd_Even, J8 Conn_02x03_Odd_Even, J9 Conn_02x03_Odd_Even, SW1 DSWB02LHGETB, U1 RT5752BHGJ5, U10 RQ12000160, U12 TMUX1574DYYR, U2 TLV803SDBZR, U3 RQ12000160, U4 ADS1115IDGSR, U5 RP2040, U6 RQ12000160, U7 ADS1115IDGSR, U8 FT2232HL, U9 93LC56BT-I

Commit message: Final commit
Parts:
- removed the C11 at (125.4, 91.3)
- removed the C13 at (127.3, 91.3)
- removed the C74 at (123.6, 76.7)
- removed the C75 at (115.4, 83.7)
- removed the C77 at (121.6, 76.8)
- removed C82, C84, C86, C87, C89, C90, C92, C93: 0.1uF, Capacitor_SMD:C_0201_0603Metric_Pad0.64x0.40mm_HandSolder
- removed C85, C88, C91: 1uF, Capacitor_SMD:C_0402_1005Metric_Pad0.74x0.62mm_HandSolder
- removed L9: HCB1005KF-121T20, Resistor_SMD:R_0402_1005Metric_Pad0.72x0.64mm_HandSolder
- removed the R14 at (128.7, 93.2)
- removed the R15 at (128.7, 92.4)
- removed the R24 at (150.0, 108.0)
- removed the R29 at (155.8, 105.7)
- removed the R46 at (128.7, 90.6)
- removed the R47 at (128.7, 91.4)
- removed the R48 at (150.5, 91.6)
- removed the R49 at (150.5, 90.8)
- removed the R5 at (115.5, 89.7)
- removed the R50 at (150.5, 93.1)
- removed the R51 at (150.5, 92.3)
- removed the R55 at (142.5, 93.5)
- removed R56: 10k, Resistor_SMD:R_0201_0603Metric_Pad0.64x0.40mm_HandSolder
- removed R65: 0, Resistor_SMD:R_0201_0603Metric_Pad0.64x0.40mm_HandSolder
- removed R67, R68, R69, R72, R73, R74, R75: 240, Resistor_SMD:R_0201_0603Metric_Pad0.64x0.40mm_HandSolder
- removed TP10, TP9: TestPoint, TestPoint:TestPoint_Pad_D1.0mm
- added C34: 22uF, Capacitor_SMD:C_0603_1608Metric_Pad1.08x0.95mm_HandSolder, B.Cu at (123.5, 93.1)
- added R19: 10k, Resistor_SMD:R_0201_0603Metric_Pad0.64x0.40mm_HandSolder, F.Cu at (115.5, 89.7)
- added R26: 10k, Resistor_SMD:R_0201_0603Metric_Pad0.64x0.40mm_HandSolder, F.Cu at (154.4, 107.4)
- added R32: 10k, Resistor_SMD:R_0201_0603Metric_Pad0.64x0.40mm_HandSolder, B.Cu at (142.5, 93.5)
- added R34: 10k, Resistor_SMD:R_0201_0603Metric_Pad0.64x0.40mm_HandSolder, B.Cu at (138.2, 93.5)
- added R37: 10k, Resistor_SMD:R_0201_0603Metric_Pad0.64x0.40mm_HandSolder, F.Cu at (155.4, 106.1)
- added R39: 10k, Resistor_SMD:R_0201_0603Metric_Pad0.64x0.40mm_HandSolder, F.Cu at (152.7, 98.9)
- added R54: 100, Resistor_SMD:R_0201_0603Metric_Pad0.64x0.40mm_HandSolder, F.Cu at (133.3, 110.4)
- added RN1: 30Ω, 2D02WGJ0300TCE:RES-ARRAY-SMD_0402-4P-L1.0-W1.0-BL, F.Cu at (128.7, 91.0)
- added RN2: 10kΩ, FRA044RJ103 TS:RES-ARRAY-SMD_0804-8P-L2.0-W1.0-BL, F.Cu at (149.8, 92.0)
- added RN3: 30Ω, 2D02WGJ0300TCE:RES-ARRAY-SMD_0402-4P-L1.0-W1.0-BL, F.Cu at (128.7, 92.7)
- J13: value PH-2A -> 1.0-3PWB; footprint Connector_JST:JST_PH_B2B-PH-K_1x02_P2.00mm_Vertical -> 1.0-3PWB:1.0-3PWB; moved to B.Cu
- R38: value 240 -> 10k
- R53: value 10k -> 100; moved to F.Cu
- moved J13 51.0 mm to (158.1, 111.5), turned to -90 degrees
- moved R53 22.6 mm to (133.3, 109.6), turned to 0 degrees
- moved R38 21.8 mm to (140.8, 88.3), turned to 180 degrees
- moved R25 3.73 mm to (150.0, 108.0)
- renumbered C76 to C1, C35 to C10, C45 to C11, C46 to C12, C50 to C13, C1 to C14, C2 to C15, C17 to C16, C32 to C17, C52 to C18, C31 to C19, C54 to C2, C51 to C20, C15 to C21, C16 to C22, C6 to C23, C7 to C24, C78 to C25, C18 to C26, C3 to C27, C19 to C28, C4 to C29, C66 to C3, C8 to C30, C5 to C31, C71 to C32, C72 to C33, C44 to C35, C42 to C36, C43 to C37, C40 to C38, C73 to C39, C36 to C4, C68 to C40, C12 to C41, C14 to C42, C83 to C43, C41 to C44, C69 to C45, C56 to C46, C38 to C47, C57 to C48, C70 to C49, C49 to C5, C39 to C50, C58 to C51, C37 to C52, C63 to C53, C64 to C54, C33 to C55, C59 to C56, C34 to C57, C60 to C58, C61 to C59, C53 to C6, C62 to C60, C47 to C61, C9 to C62, C48 to C63, C30 to C64, C27 to C65, C10 to C66, C28 to C67, C20 to C68, C21 to C69, C55 to C7, C22 to C70, C23 to C71, C24 to C72, C25 to C73, C26 to C74, C29 to C75, C81 to C76, C80 to C77, C65 to C8, C67 to C9, IC2 to IC1, IC1 to IC2, IC5 to IC3, IC3 to IC5, J7 to J10, J10 to J11, J4 to J2, J5 to J3, J2 to J4, J3 to J5, J8 to J7, J11 to J8, L6 to L5, L7 to L6, L8 to L7, L5 to L8, R37 to R1, R40 to R10, R43 to R11, R44 to R12, R19 to R13, R20 to R14, R31 to R15, R33 to R16, R10 to R17, R11 to R18, R41 to R2, R7 to R20, R63 to R21, R60 to R22, R58 to R23, R64 to R24, R36 to R27, R8 to R28, R4 to R29, R42 to R3, R35 to R30, R28 to R31, R26 to R33, R27 to R35, R71 to R36, R45 to R4, R59 to R40, R52 to R41, R13 to R42, R62 to R43, R70 to R44, R32 to R45, R22 to R46, R3 to R47, R9 to R48, R61 to R49, R16 to R5, R18 to R50, R17 to R51, R6 to R52, R2 to R55, R21 to R6, R30 to R7, R34 to R8, R39 to R9, TP3 to TP1, TP12 to TP2, U4 to U1, U5 to U10, U12 to U11, U7 to U2, U1 to U4, U9 to U5, U10 to U6, U8 to U7, U6 to U8, U2 to U9
Connections:
- C10 pad 1: Net-(C35-Pad1) -> Net-(U1-AIN0)
- C11 pad 1: Net-(C36-Pad1) -> Net-(U1-AIN1)
- C12 pad 1: Net-(C46-Pad1) -> Net-(U1-AIN2)
- C13 pad 1: Net-(C49-Pad1) -> Net-(U1-AIN3)
- C2 pad 1: Net-(C54-Pad1) -> Net-(U2-AIN1)
- C2 pad 2: Net-(C53-Pad1) -> Net-(U2-AIN0)
- C3 pad 1: Net-(C66-Pad1) -> Net-(U2-AIN3)
- C3 pad 2: Net-(C65-Pad1) -> Net-(U2-AIN2)
- C39 pad 1: Net-(U10-OSC2) -> CLK12M
- C4 pad 1: Net-(C36-Pad1) -> Net-(U1-AIN1)
- C4 pad 2: Net-(C35-Pad1) -> Net-(U1-AIN0)
- C5 pad 1: Net-(C49-Pad1) -> Net-(U1-AIN3)
- C5 pad 2: Net-(C46-Pad1) -> Net-(U1-AIN2)
- C6 pad 1: Net-(C53-Pad1) -> Net-(U2-AIN0)
- C7 pad 1: Net-(C54-Pad1) -> Net-(U2-AIN1)
- C8 pad 1: Net-(C65-Pad1) -> Net-(U2-AIN2)
- C9 pad 1: Net-(C66-Pad1) -> Net-(U2-AIN3)
- IC4 pad 16: SPI0_CS_N -> Net-(IC4-PB20C)
- IC4 pad 27: unconnected-(IC4-PT12D-Pad27) -> SPI0_CS_N
- J13 pad 1: VBUS_EXT -> Net-(J13-Pad1)
- R10 pad 2: Net-(C54-Pad1) -> Net-(U2-AIN1)
- R11 pad 2: Net-(C65-Pad1) -> Net-(U2-AIN2)
- R12 pad 2: Net-(C66-Pad1) -> Net-(U2-AIN3)
- R13 pad 2: Net-(C35-Pad1) -> Net-(U1-AIN0)
- R14 pad 2: Net-(C36-Pad1) -> Net-(U1-AIN1)
- R15 pad 2: Net-(C46-Pad1) -> Net-(U1-AIN2)
- R16 pad 2: Net-(C49-Pad1) -> Net-(U1-AIN3)
- R25 pad 2: SPI0_CS_N -> SPI0_MISO
- R38 pad 1: Net-(C35-Pad1) -> +3.3V_FT2232H
- R38 pad 2: Net-(U4-AIN0) -> Net-(U5-CS)
- R53 pad 1: +3.3V_FT2232H -> Net-(J13-Pad1)
- R53 pad 2: Net-(U8-EECS) -> Net-(U10-GPIO8)
- R9 pad 2: Net-(C53-Pad1) -> Net-(U2-AIN0)
- U1 pad 4: Net-(U4-AIN0) -> Net-(U1-AIN0)
- U1 pad 5: Net-(U4-AIN1) -> Net-(U1-AIN1)
- U1 pad 6: Net-(U4-AIN2) -> Net-(U1-AIN2)
- U1 pad 7: Net-(U4-AIN3) -> Net-(U1-AIN3)
- U10 pad 11: unconnected-(U5-GPIO8-Pad11) -> Net-(U10-GPIO8)
- U10 pad 12: unconnected-(U5-GPIO9-Pad12) -> Net-(U10-GPIO9)
- U10 pad 27: Net-(U5-GPIO16) -> unconnected-(U10-GPIO16-Pad27)
- U10 pad 28: Net-(U5-GPIO17) -> unconnected-(U10-GPIO17-Pad28)
- U2 pad 4: Net-(U7-AIN0) -> Net-(U2-AIN0)
- U2 pad 5: Net-(U7-AIN1) -> Net-(U2-AIN1)
- U2 pad 6: Net-(U7-AIN2) -> Net-(U2-AIN2)
- U2 pad 7: Net-(U7-AIN3) -> Net-(U2-AIN3)
- U5 pad 5: Net-(U8-EECS) -> Net-(U5-CS)
- U6 pad 3: Net-(U10-OSC2) -> CLK12M
- U7 pad 3: Net-(U10-OSC2) -> CLK12M
- U7 pad 63: Net-(U8-EECS) -> Net-(U5-CS)
Routing:
- net VBUS_EXT: track 61.6 -> 0.00 mm, vias 4 -> 0
- net Net-(J13-Pad1): track 0.00 -> 30.7 mm, vias 0 -> 3
- net Net-(J13-Pad3): track 0.00 -> 30.6 mm, vias 0 -> 3
- net SPI0_CS_N: track 14.0 -> 26.9 mm
- net CLK12M: track 24.6 -> 36.3 mm
- net Net-(U10-OSC2): track 11.1 -> 0.00 mm
- net Net-(U2-AIN3): track 0.00 -> 9.97 mm
- net Net-(U1-AIN3): track 0.00 -> 9.76 mm
- net Net-(U1-AIN0): track 0.00 -> 9.63 mm
- net Net-(U2-AIN0): track 0.00 -> 9.56 mm
- net Net-(U1-AIN1): track 0.00 -> 8.58 mm
- net Net-(U7-AIN0): track 8.37 -> 0.00 mm
- net Net-(U4-AIN3): track 8.33 -> 0.00 mm
- net Net-(U2-AIN2): track 0.00 -> 8.27 mm
- net Net-(U1-AIN2): track 0.00 -> 8.09 mm
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- removed copper zone on B.Cu, net VBUS_EXT
- removed copper zone on In4.Cu, net VBUS_EXT
Other:
- board text added: "SWDCLK GND SWDIO"
- board text removed: "+5V GND"
- board text removed: "RP2040 SWD"

Commit message: V2 commit
Parts:
- removed the G*** at (121.2, 109.1)
- added C31: 0.01uF, Capacitor_SMD:C_0201_0603Metric_Pad0.64x0.40mm_HandSolder, B.Cu at (134.3, 72.3)
- added C32: 1000pF, Capacitor_SMD:C_0201_0603Metric, B.Cu at (137.6, 73.4)
- added G***: LOGO, LOGO:kana_neko, F.Cu at (115.0, 85.4)
- added R26: 0, Resistor_SMD:R_0201_0603Metric_Pad0.64x0.40mm_HandSolder, B.Cu at (134.3, 71.6)
- moved C33 2.96 mm to (126.0, 93.1), turned to -90 degrees
- moved C36 1.04 mm to (124.5, 93.1), turned to -90 degrees
- moved L3 1.01 mm to (128.3, 93.2), turned to 90 degrees
- moved G*** 0.68 mm to (137.9, 99.4)
- renumbered C31 to C33, C32 to C34, C33 to C35, C34 to C36, C35 to C37, C36 to C38, C37 to C39, C38 to C40, C39 to C41, C40 to C42, C41 to C43, C42 to C44, C43 to C45, C44 to C46, C45 to C47, C46 to C48, C47 to C49, C48 to C50, C49 to C51, C50 to C52, C51 to C53, C52 to C54, C53 to C55, C54 to C56, C55 to C57, C56 to C58, C57 to C59, C58 to C60, C59 to C61, C60 to C62, C61 to C63, C62 to C64, C63 to C65, C64 to C66, C65 to C67, C66 to C68, C67 to C69, C68 to C70, C69 to C71, C70 to C72, C71 to C73, C72 to C74, C73 to C75, C74 to C76, C75 to C77, C76 to C78, C77 to C79, R26 to R27, R27 to R28, R28 to R29, R29 to R30, R30 to R31, R31 to R32, R32 to R33, R33 to R34, R34 to R35, R35 to R36, R36 to R37, R37 to R38, R38 to R39, R39 to R40, R40 to R41, R41 to R42, R42 to R43, R43 to R44, R44 to R45, R45 to R46, R46 to R47, R47 to R48, R48 to R49, R49 to R50, R50 to R51, R51 to R52, R52 to R53, R53 to R54, R54 to R55, R55 to R56
Connections:
- C30 pad 2: GND -> TMPGND
- IC3 pad 2: GND -> TMPGND
- IC3 pad 5: GND -> TMPGND
Routing:
- net GND: track 1281.1 -> 1299.1 mm, vias 385 -> 376
- net TMPGND: track 0.00 -> 11.9 mm
- net +3.3V: track 20.8 -> 18.1 mm
- net +3.3V_ADC: track 93.5 -> 92.7 mm
- added copper zone on B.Cu, net Net-(U4-SW)
- added copper zone on B.Cu, net TMPGND
Other:
- board text added: "DBGP_CLK GND DBGP_IO"
- board text added: "KANAYUI-SX01A"
- board text removed: "JLCJLCJLCJLC"
