File: FlexLogicMini_EVB.kicad_sch (KiCad schematic)
At the start: 205 parts, among them IC1 MT9700, IC2 SL2.1s, IC3 W25Q16JVUXIQ, IC4 LCMXO2-1200HC-4SG32I, IC5 MTS4P, J1 GT-USB-7010ASV, J10 Conn_01x04, J11 Conn_02x03_Odd_Even, J12 1.0-3PWB, J13 PH-2A, J2 WJ126V-5.0-2P, J3 WJ126V-5.0-2P, J4 WJ126V-5.0-2P, J5 WJ126V-5.0-2P, J6 Conn_02x03_Odd_Even, J7 Conn_02x03_Odd_Even, J8 Conn_02x03_Odd_Even, J9 Conn_02x03_Odd_Even, SW1 DSWB02LHGETB, U1 RT5752BHGJ5, U10 RQ12000160, U2 TLV803SDBZR, U3 RQ12000160, U4 ADS1115IDGSR, U5 RP2040, U6 RQ12000160, U7 ADS1115IDGSR, U8 FT2232HL, U9 93LC56BT-I

Commit message: Final commit
Parts:
- removed C11, C13, C75, C77, C82, C84, C86, C87, C89, C90, C92, C93: 0.1uF, Capacitor_SMD:C_0201_0603Metric_Pad0.64x0.40mm_HandSolder, symbol Device:C_Small
- removed C74, C85, C88, C91: 1uF, Capacitor_SMD:C_0402_1005Metric_Pad0.74x0.62mm_HandSolder, symbol Device:C_Small
- removed J13: PH-2A, Connector_JST:JST_PH_B2B-PH-K_1x02_P2.00mm_Vertical, symbol Connector_Generic:Conn_02x01
- removed L9: HCB1005KF-121T20, Resistor_SMD:R_0402_1005Metric_Pad0.72x0.64mm_HandSolder, symbol hcb1005kf-121t20:HCB1005KF-121T20
- removed R14, R15, R46, R47: 30, Resistor_SMD:R_0201_0603Metric_Pad0.64x0.40mm_HandSolder, symbol Device:R
- removed R24, R29, R48, R49, R50, R51, R55, R56: 10k, Resistor_SMD:R_0201_0603Metric_Pad0.64x0.40mm_HandSolder, symbol Device:R
- removed R5: 4.7k, Resistor_SMD:R_0201_0603Metric_Pad0.64x0.40mm_HandSolder, symbol Device:R
- removed R65: 0, Resistor_SMD:R_0201_0603Metric_Pad0.64x0.40mm_HandSolder, symbol Device:R
- removed R67, R68, R69, R72, R73, R74, R75: 240, Resistor_SMD:R_0201_0603Metric_Pad0.64x0.40mm_HandSolder, symbol Device:R
- removed TP10, TP9: TestPoint, TestPoint:TestPoint_Pad_D1.0mm, symbol Connector:TestPoint
- added C34: 22uF, Capacitor_SMD:C_0603_1608Metric_Pad1.08x0.95mm_HandSolder, symbol Device:C_Small
- added J13: 1.0-3PWB, 1.0-3PWB:1.0-3PWB, symbol 1.0-3PWB:1.0-3PWB
- added R19, R26, R32, R34, R37, R39: 10k, Resistor_SMD:R_0201_0603Metric_Pad0.64x0.40mm_HandSolder, symbol Device:R
- added R54: 100, Resistor_SMD:R_0201_0603Metric_Pad0.64x0.40mm_HandSolder, symbol Device:R
- added RN1, RN3: 30Ω, 2D02WGJ0300TCE:RES-ARRAY-SMD_0402-4P-L1.0-W1.0-BL, symbol 2D02WGJ0300TCE:2D02WGJ0300TCE
- added RN2: 10kΩ, FRA044RJ103 TS:RES-ARRAY-SMD_0804-8P-L2.0-W1.0-BL, symbol FRA044RJ103 TS:FRA044RJ103 TS
- IC1: renamed from IC2; DESCRIPTION USB2.0 HUB -> (none)
- IC2: renamed from IC1; DESCRIPTION Current-Limited Power-Distribution Switch -> (none)
- R38: value 240 -> 10k; JLCPCB C320776 -> C106225; MANUFACTURER_PART_NUMBER RC-01W241JT -> RC0201FR-0710KL
- R53: value 10k -> 100; JLCPCB C106225 -> C106229; MANUFACTURER_PART_NUMBER RC0201FR-0710KL -> RC0201JR-07100RL
- renumbered C76 to C1, C35 to C10, C45 to C11, C46 to C12, C50 to C13, C1 to C14, C2 to C15, C17 to C16, C32 to C17, C52 to C18, C31 to C19, C54 to C2, C51 to C20, C15 to C21, C16 to C22, C6 to C23, C7 to C24, C78 to C25, C18 to C26, C3 to C27, C19 to C28, C4 to C29, C66 to C3, C8 to C30, C5 to C31, C71 to C32, C72 to C33, C44 to C35, C42 to C36, C43 to C37, C40 to C38, C73 to C39, C36 to C4, C68 to C40, C12 to C41, C14 to C42, C83 to C43, C41 to C44, C69 to C45, C56 to C46, C38 to C47, C57 to C48, C70 to C49, C49 to C5, C39 to C50, C58 to C51, C37 to C52, C63 to C53, C64 to C54, C33 to C55, C59 to C56, C34 to C57, C60 to C58, C61 to C59, C53 to C6, C62 to C60, C47 to C61, C9 to C62, C48 to C63, C30 to C64, C27 to C65, C10 to C66, C28 to C67, C20 to C68, C21 to C69, C55 to C7, C22 to C70, C23 to C71, C24 to C72, C25 to C73, C26 to C74, C29 to C75, C81 to C76, C65 to C8, C67 to C9, IC5 to IC3, IC3 to IC5, J7 to J10, J10 to J11, J4 to J2, J5 to J3, J2 to J4, J3 to J5, J8 to J7, J11 to J8, L6 to L5, L7 to L6, L8 to L7, L5 to L8, R37 to R1, R40 to R10, R43 to R11, R44 to R12, R19 to R13, R20 to R14, R31 to R15, R33 to R16, R10 to R17, R11 to R18, R41 to R2, R7 to R20, R63 to R21, R60 to R22, R58 to R23, R64 to R24, R36 to R27, R8 to R28, R4 to R29, R42 to R3, R35 to R30, R28 to R31, R26 to R33, R27 to R35, R71 to R36, R45 to R4, R59 to R40, R52 to R41, R13 to R42, R62 to R43, R70 to R44, R32 to R45, R22 to R46, R3 to R47, R9 to R48, R61 to R49, R16 to R5, R18 to R50, R17 to R51, R6 to R52, R2 to R55, R21 to R6, R30 to R7, R34 to R8, R39 to R9, TP3 to TP1, TP12 to TP2, U4 to U1, U5 to U10, U7 to U2, U1 to U4, U9 to U5, U10 to U6, U8 to U7, U6 to U8, U2 to U9
Connections:
- net +3.3V: now also C34.1
- net +3.3V_D: now also R26.1, R37.1, R39.1
- net +3.3V_FT2232H: now also R38.1, R32.1, R34.1, RN2.5, RN2.6, RN2.7, RN2.8; no longer R53.1
- net CLK12M: now also C39.1, U6.3 (OSC2), U7.3 (OSCO)
- net CTS_N_PIN: now also RN2.1
- net FT2232H_N: now also RN1.3
- net FT2232H_P: now also RN1.4
- net GND: now also C34.2, J13.2, J13.4, J13.5
- net RP2040_N: now also RN3.3
- net RP2040_P: now also RN3.4
- net RTS_N_PIN: now also RN2.2
- net RXD_PIN: now also RN2.3
- net SPI0_CS_N: now also IC4.27 (PT12D), R39.2; no longer IC4.16 (PB20C), R25.2
- net SPI0_MISO: now also R25.2
- net SPI0_MOSI: now also R37.2
- net TXD_PIN: now also RN2.4
- net USB_FT2232H+: now also RN1.1
- net USB_FT2232H-: now also RN1.2
- net USB_MCU+: now also RN3.1
- net USB_MCU-: now also RN3.2
- net at U1.7 (AIN3): now also C13.1, C5.1, R16.2
- net at U1.6 (AIN2): now also C12.1, C5.2, R15.2
- net at U1.4 (AIN0): now also C10.1, C4.2, R13.2; no longer R38.2
- net at U1.5 (AIN1): now also C11.1, C4.1, R14.2
- net at C14.1, D1.1 (A1), J1.A4B9 (VBUS)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: now also R19.1
- net at C3.2, C8.1, R11.2: now also U2.6 (AIN2)
- net at U5.5 (CS), U7.63 (EECS): now also R38.2; no longer R53.2
- net at U2.7 (AIN3): now also C3.1, C9.1, R12.2
- net at R36.2, U5.3 (DI), U7.61 (EEDATA): now also R34.2
- net at C2.2, C6.1, R9.2: now also U2.4 (AIN0)
- net at U10.11 (GPIO8): now also R53.2
- net at U10.12 (GPIO9): now also R54.2
- net at C2.1, C7.1, R10.2: now also U2.5 (AIN1)
- net at D2.2 (A): now also R19.2
- net at R36.1, U5.1 (DO): now also R32.2
- new net: J13.1, R53.1
- new net: J13.3, R54.1
- new net: IC4.16 (PB20C), R26.2
- no-connect marks 50 -> 49
Other:
- note added: "DBGP_SWCLK GND DBGP_SWDIO"
- note added: "SWD Debug Probe(PIO0)"
- note removed: "External Power Pinheader"
- moved on the sheet: R31, R33, R35

Commit message: V2 commit
Parts:
- added C31: 0.01uF, Capacitor_SMD:C_0201_0603Metric_Pad0.64x0.40mm_HandSolder, symbol Device:C_Small
- added C32: 1000pF, Capacitor_SMD:C_0201_0603Metric, symbol Device:C_Small
- added R26: 0, Resistor_SMD:R_0201_0603Metric_Pad0.64x0.40mm_HandSolder, symbol Device:R
- renumbered C31 to C33, C32 to C34, C33 to C35, C34 to C36, C35 to C37, C36 to C38, C37 to C39, C38 to C40, C39 to C41, C40 to C42, C41 to C43, C42 to C44, C43 to C45, C44 to C46, C45 to C47, C46 to C48, C47 to C49, C48 to C50, C49 to C51, C50 to C52, C51 to C53, C52 to C54, C53 to C55, C54 to C56, C55 to C57, C56 to C58, C57 to C59, C58 to C60, C59 to C61, C60 to C62, C61 to C63, C62 to C64, C63 to C65, C64 to C66, C65 to C67, C66 to C68, C67 to C69, C68 to C70, C69 to C71, C70 to C72, C71 to C73, C72 to C74, C73 to C75, C74 to C76, C75 to C77, C76 to C78, R26 to R27, R27 to R28, R28 to R29, R29 to R30, R30 to R31, R31 to R32, R32 to R33, R33 to R34, R34 to R35, R35 to R36, R36 to R37, R37 to R38, R38 to R39, R39 to R40, R40 to R41, R41 to R42, R42 to R43, R43 to R44, R44 to R45, R45 to R46, R46 to R47, R47 to R48, R48 to R49, R49 to R50, R50 to R51, R51 to R52, R52 to R53, R53 to R54, R54 to R55, R55 to R56
Connections:
- net GND: now also C31.2, C32.1, R26.1; no longer C30.2, IC3.2 (GND), IC3.5 (EP)
- new net TMPGND: C30.2, C31.1, C32.2, IC3.2 (GND), IC3.5 (EP), R26.2
Other:
- moved on the sheet: C30, IC3

Commit message: V3 commit
Parts:
- removed C31: 0.01uF, Capacitor_SMD:C_0201_0603Metric_Pad0.64x0.40mm_HandSolder, symbol Device:C_Small
- removed C34, C40, C66, C77, C78: 0.1uF, Capacitor_SMD:C_0201_0603Metric_Pad0.64x0.40mm_HandSolder, symbol Device:C_Small
- removed R27, R40: 10k, Resistor_SMD:R_0201_0603Metric_Pad0.64x0.40mm_HandSolder, symbol Device:R
- removed R36: 4.7k, Resistor_SMD:R_0201_0603Metric_Pad0.64x0.40mm_HandSolder, symbol Device:R
- removed R52: 2.2k, Resistor_SMD:R_0201_0603Metric_Pad0.64x0.40mm_HandSolder, symbol Device:R
- removed R55: 100, Resistor_SMD:R_0201_0603Metric_Pad0.64x0.40mm_HandSolder, symbol Device:R
- added C33: 33pF, Capacitor_SMD:C_0402_1005Metric, symbol Device:C_Small
- added C36, C42: 0.1uF, Capacitor_SMD:C_0402_1005Metric, symbol Device:C_Small
- added C68: 1uF, Capacitor_SMD:C_0402_1005Metric, symbol Device:C_Small
- added R30: 2.2k, Resistor_SMD:R_0402_1005Metric, symbol Device:R
- added R37: 10k, Resistor_SMD:R_0402_1005Metric, symbol Device:R
- added R44, R53: 100, Resistor_SMD:R_0402_1005Metric, symbol Device:R
- C1, C10, C11, C12, C13, C14, C19, C20, C23, C25, C30, C37, C38, C43, C44, C45, C46, C47, C48, C49, C50, C51, C52, C53, C54, C56, C58, C59, C6, C60, C62, C64, C7, C71, C72, C73, C74, C75, C76, C8, C9: footprint Capacitor_SMD:C_0201_0603Metric_Pad0.64x0.40mm_HandSolder -> Capacitor_SMD:C_0402_1005Metric; JLCPCB C76939 -> C307331; MANUFACTURER_PART_NUMBER GRM033R61E104KE14D -> CL05B104KB54PNC; 耐圧 25V -> 50V
- C15, C16, C21, C22, C24: footprint Capacitor_SMD:C_0402_1005Metric_Pad0.74x0.62mm_HandSolder -> Capacitor_SMD:C_0402_1005Metric
- C17, C18: footprint Capacitor_SMD:C_0201_0603Metric_Pad0.64x0.40mm_HandSolder -> Capacitor_SMD:C_0402_1005Metric; JLCPCB C285010 -> C15195; MANUFACTURER_PART_NUMBER 0201B103K250NT -> CL05B103KB5NNNC; 耐圧 25V -> 50V
- C2, C3, C4, C5: footprint Capacitor_SMD:C_0402_1005Metric_Pad0.74x0.62mm_HandSolder -> Capacitor_SMD:C_0402_1005Metric; JLCPCB C2887021 -> C52923; MANUFACTURER_PART_NUMBER TCC0402X5R105M6R3AT -> CL05A105KA5NQNC; 耐圧 6.3V -> 25V
- C26, C28, C63: value 30pF -> 33pF; footprint Capacitor_SMD:C_0201_0603Metric_Pad0.64x0.40mm_HandSolder -> Capacitor_SMD:C_0402_1005Metric; JLCPCB C5142545 -> C1562; MANUFACTURER_PART_NUMBER TCC0201COG300J500ZT -> 0402CG330J500NT
- C32: value 1000pF -> 0.1uF; footprint Capacitor_SMD:C_0201_0603Metric -> Capacitor_SMD:C_0402_1005Metric; JLCPCB C5142559 -> C307331; MANUFACTURER_PART_NUMBER TCC0201X7R102K500ZT -> CL05B104KB54PNC
- C35, C41, C65: value 30pF -> 0.1uF; footprint Capacitor_SMD:C_0201_0603Metric_Pad0.64x0.40mm_HandSolder -> Capacitor_SMD:C_0402_1005Metric; JLCPCB C5142545 -> C307331; MANUFACTURER_PART_NUMBER TCC0201COG300J500ZT -> CL05B104KB54PNC
- C39, C61: value 0.1uF -> 33pF; footprint Capacitor_SMD:C_0201_0603Metric_Pad0.64x0.40mm_HandSolder -> Capacitor_SMD:C_0402_1005Metric; JLCPCB C76939 -> C1562; MANUFACTURER_PART_NUMBER GRM033R61E104KE14D -> 0402CG330J500NT; 耐圧 25V -> 50V
- C40: renamed from C42; footprint Capacitor_SMD:C_0402_1005Metric_Pad0.74x0.62mm_HandSolder -> Capacitor_SMD:C_0402_1005Metric
- C55, C67: value 0.1uF -> 1uF; footprint Capacitor_SMD:C_0201_0603Metric_Pad0.64x0.40mm_HandSolder -> Capacitor_SMD:C_0402_1005Metric; JLCPCB C76939 -> C52923; MANUFACTURER_PART_NUMBER GRM033R61E104KE14D -> CL05A105KA5NQNC
- C57, C69, C70: value 1uF -> 0.1uF; footprint Capacitor_SMD:C_0402_1005Metric_Pad0.74x0.62mm_HandSolder -> Capacitor_SMD:C_0402_1005Metric; JLCPCB C2887021 -> C307331; MANUFACTURER_PART_NUMBER TCC0402X5R105M6R3AT -> CL05B104KB54PNC; 耐圧 6.3V -> 50V
- C66: renamed from C68; footprint Capacitor_SMD:C_0201_0603Metric_Pad0.64x0.40mm_HandSolder -> Capacitor_SMD:C_0402_1005Metric; JLCPCB C76939 -> C307331; MANUFACTURER_PART_NUMBER GRM033R61E104KE14D -> CL05B104KB54PNC; 耐圧 25V -> 50V
- R1, R2, R3, R4, R5, R6, R7, R8: footprint Resistor_SMD:R_0201_0603Metric_Pad0.64x0.40mm_HandSolder -> Resistor_SMD:R_0402_1005Metric; JLCPCB C295786 -> C26083; MANUFACTURER_PART_NUMBER RC0201FR-071ML -> 0402WGF1004TCE; 耐電力 1/20W -> 1/16W
- R10, R11, R12, R13, R14, R15, R16, R9: value 240 -> 220; footprint Resistor_SMD:R_0201_0603Metric_Pad0.64x0.40mm_HandSolder -> Resistor_SMD:R_0402_1005Metric; JLCPCB C320776 -> C25091; MANUFACTURER_PART_NUMBER RC-01W241JT -> 0402WGF2200TCE; 耐電力 1/20W -> 1/16W
- R17, R18: footprint Resistor_SMD:R_0201_0603Metric_Pad0.64x0.40mm_HandSolder -> Resistor_SMD:R_0402_1005Metric; JLCPCB C270344 -> C25905; MANUFACTURER_PART_NUMBER 0201WMF5101TEE -> 0402WGF5101TCE; 耐電力 1/20W -> 1/16W
- R19, R22, R23, R25, R38, R39: footprint Resistor_SMD:R_0201_0603Metric_Pad0.64x0.40mm_HandSolder -> Resistor_SMD:R_0402_1005Metric; JLCPCB C106225 -> C25744; MANUFACTURER_PART_NUMBER RC0201FR-0710KL -> 0402WGF1002TCE; 耐電力 1/20W -> 1/16W
- R20: footprint Resistor_SMD:R_0201_0603Metric_Pad0.64x0.40mm_HandSolder -> Resistor_SMD:R_0402_1005Metric; Field7 (none) -> 1/16W; JLCPCB C367600 -> C3017490; MANUFACTURER_PART_NUMBER WR02X362JAL -> SCR0402J3K6
- R21, R24, R31, R51: footprint Resistor_SMD:R_0201_0603Metric_Pad0.64x0.40mm_HandSolder -> Resistor_SMD:R_0402_1005Metric; JLCPCB C171950 -> C25879; MANUFACTURER_PART_NUMBER WR02X222JAL -> 0402WGF2201TCE; 耐電力 1/20W -> 1/16W
- R26: value 0 -> 10k; footprint Resistor_SMD:R_0201_0603Metric_Pad0.64x0.40mm_HandSolder -> Resistor_SMD:R_0402_1005Metric; JLCPCB (none) -> C25744; MANUFACTURER_PART_NUMBER (none) -> 0402WGF1002TCE; 耐電力 1/20W -> 1/16W
- R27: renamed from R28; footprint Resistor_SMD:R_0201_0603Metric_Pad0.64x0.40mm_HandSolder -> Resistor_SMD:R_0402_1005Metric; JLCPCB C270346 -> C25900; MANUFACTURER_PART_NUMBER 0201WMF4701TEE -> 0402WGF4701TCE; 耐電力 1/20W -> 1/16W
- R28: renamed from R29; footprint Resistor_SMD:R_0201_0603Metric_Pad0.64x0.40mm_HandSolder -> Resistor_SMD:R_0402_1005Metric; JLCPCB C473469 -> C25768; MANUFACTURER_PART_NUMBER 0201WMF2202TEE -> 0402WGF2202TCE; 耐電力 1/20W -> 1/16W
- R29: renamed from R30; footprint Resistor_SMD:R_0201_0603Metric_Pad0.64x0.40mm_HandSolder -> Resistor_SMD:R_0402_1005Metric; JLCPCB C304505 -> C25741; MANUFACTURER_PART_NUMBER RC-01W104JT -> 0402WGF1003TCE; 耐電力 1/20W -> 1/16W
- R32: value 2.2k -> 10k; footprint Resistor_SMD:R_0201_0603Metric_Pad0.64x0.40mm_HandSolder -> Resistor_SMD:R_0402_1005Metric; JLCPCB C171950 -> C25744; MANUFACTURER_PART_NUMBER WR02X222JAL -> 0402WGF1002TCE; 耐電力 1/20W -> 1/16W
- R33, R35: value 10k -> 4.7k; footprint Resistor_SMD:R_0201_0603Metric_Pad0.64x0.40mm_HandSolder -> Resistor_SMD:R_0402_1005Metric; JLCPCB C106225 -> C25900; MANUFACTURER_PART_NUMBER RC0201FR-0710KL -> 0402WGF4701TCE; 耐電力 1/20W -> 1/16W
- R34: value 4.7k -> 10k; footprint Resistor_SMD:R_0201_0603Metric_Pad0.64x0.40mm_HandSolder -> Resistor_SMD:R_0402_1005Metric; JLCPCB C270346 -> C25744; MANUFACTURER_PART_NUMBER 0201WMF4701TEE -> 0402WGF1002TCE; 耐電力 1/20W -> 1/16W
- R36: renamed from R37; footprint Resistor_SMD:R_0201_0603Metric_Pad0.64x0.40mm_HandSolder -> Resistor_SMD:R_0402_1005Metric; JLCPCB C171950 -> C25879; MANUFACTURER_PART_NUMBER WR02X222JAL -> 0402WGF2201TCE; 耐電力 1/20W -> 1/16W
- R40: renamed from R41; value 30 -> 33; footprint Resistor_SMD:R_0201_0603Metric_Pad0.64x0.40mm_HandSolder -> Resistor_SMD:R_0402_1005Metric; JLCPCB C320826 -> C25105; MANUFACTURER_PART_NUMBER RC-01W30R0FT -> 0402WGF330JTCE; 耐電力 1/20W -> 1/16W
- R41: renamed from R42; footprint Resistor_SMD:R_0201_0603Metric_Pad0.64x0.40mm_HandSolder -> Resistor_SMD:R_0402_1005Metric; JLCPCB C270363 -> C25752; MANUFACTURER_PART_NUMBER 0201WMF1202TEE -> HGC0402R5106M100NTEJ; 耐電力 1/20W -> 1/16W
- R42: renamed from R43; footprint Resistor_SMD:R_0201_0603Metric_Pad0.64x0.40mm_HandSolder -> Resistor_SMD:R_0402_1005Metric; JLCPCB C106225 -> C25744; MANUFACTURER_PART_NUMBER RC0201FR-0710KL -> 0402WGF1002TCE; 耐電力 1/20W -> 1/16W
- R43: renamed from R44; footprint Resistor_SMD:R_0201_0603Metric_Pad0.64x0.40mm_HandSolder -> Resistor_SMD:R_0402_1005Metric; JLCPCB C106229 -> C25076; MANUFACTURER_PART_NUMBER RC0201JR-07100RL -> 0402WGF1000TCE; 耐電力 1/20W -> 1/16W
- R45: value 100 -> 33; footprint Resistor_SMD:R_0201_0603Metric_Pad0.64x0.40mm_HandSolder -> Resistor_SMD:R_0402_1005Metric; JLCPCB C106229 -> C25105; MANUFACTURER_PART_NUMBER RC0201JR-07100RL -> 0402WGF330JTCE; 耐電力 1/20W -> 1/16W
- R46, R49: value 30 -> 33; footprint Resistor_SMD:R_0201_0603Metric_Pad0.64x0.40mm_HandSolder -> Resistor_SMD:R_0402_1005Metric; JLCPCB C320826 -> C25105; MANUFACTURER_PART_NUMBER RC-01W30R0FT -> 0402WGF330JTCE; 耐電力 1/20W -> 1/16W
- R47: value 30 -> 10k; footprint Resistor_SMD:R_0201_0603Metric_Pad0.64x0.40mm_HandSolder -> Resistor_SMD:R_0402_1005Metric; JLCPCB C320826 -> C25744; MANUFACTURER_PART_NUMBER RC-01W30R0FT -> 0402WGF1002TCE; 耐電力 1/20W -> 1/16W
- R48: value 10k -> 33; footprint Resistor_SMD:R_0201_0603Metric_Pad0.64x0.40mm_HandSolder -> Resistor_SMD:R_0402_1005Metric; JLCPCB C106225 -> C25105; MANUFACTURER_PART_NUMBER RC0201FR-0710KL -> 0402WGF330JTCE; 耐電力 1/20W -> 1/16W
- R50: value 30 -> 2.2k; footprint Resistor_SMD:R_0201_0603Metric_Pad0.64x0.40mm_HandSolder -> Resistor_SMD:R_0402_1005Metric; JLCPCB C320826 -> C25879; MANUFACTURER_PART_NUMBER RC-01W30R0FT -> 0402WGF2201TCE; 耐電力 1/20W -> 1/16W
- R52: renamed from R53; footprint Resistor_SMD:R_0201_0603Metric_Pad0.64x0.40mm_HandSolder -> Resistor_SMD:R_0402_1005Metric; JLCPCB C138165 -> C11702; MANUFACTURER_PART_NUMBER RC0201FR-071KL -> 0402WGF1001TCE; 耐電力 1/20W -> 1/16W
- R54: footprint Resistor_SMD:R_0201_0603Metric_Pad0.64x0.40mm_HandSolder -> Resistor_SMD:R_0402_1005Metric; JLCPCB C106229 -> C25076; MANUFACTURER_PART_NUMBER RC0201JR-07100RL -> 0402WGF1000TCE; 耐電力 1/20W -> 1/16W
- R55: renamed from R56; footprint Resistor_SMD:R_0201_0603Metric_Pad0.64x0.40mm_HandSolder -> Resistor_SMD:R_0402_1005Metric; JLCPCB C270346 -> C25900; MANUFACTURER_PART_NUMBER 0201WMF4701TEE -> 0402WGF4701TCE; 耐電力 1/20W -> 1/16W
- renumbered C33 to C31, C36 to C34
Connections:
- net +1.1V_MCU: now also C64.1, C65.1, C67.2; no longer C67.1, C69.2
- net +3.3V_ADC: now also C42.1; no longer C44.1
- net +3.3V_A_FT2232H: now also C41.1, C53.1, C54.1; no longer C43.1, C55.1, C56.1
- net +3.3V_D: now also C35.1, C44.1, C47.1, C50.1, C55.2, C57.1, C69.1, C70.1, R26.1, R31.1, R33.1, R35.1, R39.1, R47.1, R50.1, C36.1, C68.2, R37.1; no longer C39.1, C46.1, C49.1, C54.1, C57.2, C59.1, C70.2, R32.1, R34.1, R38.1, R48.1
- net +3.3V_EXT: now also C43.1; no longer C45.1
- net +3.3V_FT2232H: now also C32.1, C49.1, C56.1, C59.1, R32.1, R34.1, R38.1; no longer C51.1, C61.1, C62.1, R33.1, R35.1, R39.1
- net CLK12M: now also C39.1; no longer C41.1
- net GND: now also C30.2, C32.2, C35.2, C55.1, C57.2, C61.1, C63.2, C67.1, C69.2, C70.2, IC3.2 (GND), IC3.5 (EP), C33.1, C36.2, C42.2, C68.1, R30.2; no longer C32.1, C35.1, C55.2, C57.1, C61.2, C63.1, C67.2, C69.1, C70.1, R26.1, R31.2
- net I2CSCL_ADC: now also R51.2
- net I2CSDA_ADC: now also R50.2; no longer R51.2
- net QSPI_SCLK: now also R46.1; no longer R47.1
- net RESET_N: now also R47.2, R48.1; no longer R48.2, R49.1
- net SPI0_CLK: now also R49.2; no longer R50.2
- net SPI0_CS_N: now also R39.2
- net SPI0_MOSI: now also R37.2; no longer R38.2
- net TCK_FPGA: now also R30.1; no longer R31.1
- net TMS_FPGA: now also R31.2; no longer R32.2
- net VBUS: now also C62.1; no longer C64.1
- net VCORE_FT2232H: now also C45.1, C46.1, C51.1; no longer C47.1, C50.1, C53.1
- net at U6.1 (OSC), U7.2 (OSCI): now also C33.2; no longer C35.2
- net at S1.1, S1.2: now also R48.2; no longer R49.2
- net at R45.1: now also C63.1, U8.3 (OSC2); no longer J12.3
- net at R45.2: now also U10.21 (XOUT); no longer U10.25 (SWD)
- net at U10.11 (GPIO8): now also R53.1; no longer R54.2
- net at U10.12 (GPIO9): now also R54.1
- net at U10.20 (XIN), U8.1 (OSC): now also C61.2; no longer C63.2
- net at R46.2: now also U10.52 (QSPI_SCLK); no longer U10.21 (XOUT)
- net at U10.34 (GPIO22): now also R49.1; no longer R50.1
- net at J13.1: now also R53.2; no longer R54.1
- net at J13.3: now also R54.2
- net at R34.2: now also R36.2, U5.3 (DI), U7.61 (EEDATA); no longer IC4.26 (PT15C)
- net at U5.5 (CS), U7.63 (EECS): now also R38.2; no longer R39.2
- net at R36.1, U5.1 (DO): now also R32.2; no longer R33.2
- net at IC4.16 (PB20C): now also R26.2
- net at IC4.25 (PT15D): now also R35.2
- removed net TMPGND: C30.2, C32.2, IC3.2 (GND), IC3.5 (EP), R26.2
- new net: R44.2, U10.25 (SWD)
- new net: J12.3, R44.1
- new net: IC4.26 (PT15C), R33.2
Other:
- note added: "J3とJ4の間に配置 部品面で一点アース Via禁止"
- note removed: "J3とJ4の間に配置"
