File: JTAG_Select.kicad_sch (KiCad schematic)
At the start: 2 parts, among them U12 TMUX1574DYYR

Commit message: Final commit
Parts:
- renumbered C80 to C77, U12 to U11
Changed lines of the file:
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@@
 (kicad_sch
-	(version 20250114)
+	(version 20260306)
 	(generator "eeschema")
-	(generator_version "9.0")
+	(generator_version "10.0")
 	(paper "A4")
 	(rectangle
@@
 		(mirror y)
 		(unit 1)
+		(body_style 1)
 		(exclude_from_sim no)
 		(in_bom yes)
 		(on_board yes)
+		(in_pos_files yes)
 		(dnp no)
-		(property "Reference" "C80"
+		(property "Reference" "C77"
 			(at 191.008 93.091 0)
+			(show_name no)
+			(do_not_autoplace no)
 			(effects
 				(font
@@
 		(property "Value" "0.1uF"
 			(at 192.024 96.774 0)
+			(show_name no)
+			(do_not_autoplace no)
 			(effects
 				(font
@@
 		(property "Footprint" "Capacitor_SMD:C_0201_0603Metric_Pad0.64x0.40mm_HandSolder"
 			(at 186.563 94.996 0)
+			(hide yes)
+			(show_name no)
+			(do_not_autoplace no)
 			(effects
 				(font
 					(size 1.27 1.27)
 				)
-				(hide yes)
 			)
 		)
-		(property "Datasheet" "~"
+		(property "Datasheet" ""
 			(at 186.563 94.996 0)
+			(hide yes)
+			(show_name no)
+			(do_not_autoplace no)
 			(effects
 				(font
 					(size 1.27 1.27)
 				)
-				(hide yes)
 			)
 		)
 		(property "Description" "Unpolarized capacitor, small symbol"
 			(at 186.563 94.996 0)
+			(hide yes)
+			(show_name no)
+			(do_not_autoplace no)
 			(effects
 				(font
 					(size 1.27 1.27)
 				)
-				(hide yes)
 			)
 		)
 		(property "耐圧" "25V"
 			(at 188.722 98.425 0)
+			(show_name no)
+			(do_not_autoplace no)
 			(effects
 				(font
@@
 		(property "JLCPCB" "C76939"
 			(at 186.563 94.996 0)
+			(hide yes)
+			(show_name no)
+			(do_not_autoplace no)
 			(effects
 				(font
 					(size 1.27 1.27)
 				)
-				(hide yes)
 			)
 		)
 		(property "MANUFACTURER_PART_NUMBER" "GRM033R61E104KE14D"
 			(at 186.563 94.996 0)
+			(hide yes)
+			(show_name no)
+			(do_not_autoplace no)
 			(effects
 				(font
 					(size 1.27 1.27)
 				)
-				(hide yes)
 			)
 		)
@@
 		)
 		(instances
-			(project "FT2232H_EVB"
+			(project "FlexLogicMini_EVB"
 				(path "/483d0913-2604-458a-955b-5458dee34109/5b1eb57d-d000-4da8-a3b9-023ba32e6541"
-					(reference "C80")
+					(reference "C77")
 					(unit 1)
 				)
@@
 		(mirror y)
 		(unit 1)
+		(body_style 1)
 		(exclude_from_sim no)
 		(in_bom yes)
 		(on_board yes)
+		(in_pos_files yes)
 		(dnp no)
-		(property "Reference" "#PWR0119"
+		(property "Reference" "#PWR0123"
 			(at 186.563 104.521 0)
+			(hide yes)
+			(show_name no)
+			(do_not_autoplace no)
 			(effects
 				(font
 					(size 1.27 1.27)
 				)
-				(hide yes)
 			)
 		)
 		(property "Value" "GND"
 			(at 186.563 101.981 0)
+			(show_name no)
+			(do_not_autoplace no)
 			(effects
 				(font
@@
 		(property "Footprint" ""
 			(at 186.563 98.171 0)
+			(hide yes)
+			(show_name no)
+			(do_not_autoplace no)
 			(effects
 				(font
 					(size 1.27 1.27)
 				)
-				(hide yes)
 			)
 		)
 		(property "Datasheet" ""
 			(at 186.563 98.171 0)
+			(hide yes)
+			(show_name no)
+			(do_not_autoplace no)
 			(effects
 				(font
 					(size 1.27 1.27)
 				)
-				(hide yes)
 			)
 		)
 		(property "Description" "Power symbol creates a global label with name \"GND\" , ground"
 			(at 186.563 98.171 0)
+			(hide yes)
+			(show_name no)
+			(do_not_autoplace no)
 			(effects
 				(font
 					(size 1.27 1.27)
 				)
-				(hide yes)
 			)
 		)
@@
 		)
 		(instances
-			(project "FT2232H_EVB"
+			(project "FlexLogicMini_EVB"
 				(path "/483d0913-2604-458a-955b-5458dee34109/5b1eb57d-d000-4da8-a3b9-023ba32e6541"
-					(reference "#PWR0119")
+					(reference "#PWR0123")
 					(unit 1)
 				)
@@
 		(mirror y)
 		(unit 1)
+		(body_style 1)
 		(exclude_from_sim no)
 		(in_bom yes)
 		(on_board yes)
+		(in_pos_files yes)
 		(dnp no)
-		(property "Reference" "#PWR0120"
+		(property "Reference" "#PWR0122"
 			(at 178.689 158.75 0)
+			(hide yes)
+			(show_name no)
+			(do_not_autoplace no)
 			(effects
 				(font
 					(size 1.27 1.27)
 				)
-				(hide yes)
 			)
 		)
 		(property "Value" "GND"
 			(at 178.689 155.829 0)
+			(show_name no)
+			(do_not_autoplace no)
 			(effects
 				(font
@@
 		(property "Footprint" ""
 			(at 178.689 152.4 0)
+			(hide yes)
+			(show_name no)
+			(do_not_autoplace no)
 			(effects
 				(font
 					(size 1.27 1.27)
 				)
-				(hide yes)
 			)
 		)
 		(property "Datasheet" ""
 			(at 178.689 152.4 0)
+			(hide yes)
+			(show_name no)
+			(do_not_autoplace no)
 			(effects
 				(font
 					(size 1.27 1.27)
 				)
-				(hide yes)
 			)
 		)
 		(property "Description" "Power symbol creates a global label with name \"GND\" , ground"
 			(at 178.689 152.4 0)
+			(hide yes)
+			(show_name no)
+			(do_not_autoplace no)
 			(effects
 				(font
 					(size 1.27 1.27)
 				)
-				(hide yes)
 			)
 		)
@@
 		)
 		(instances
-			(project "FT2232H_EVB"
+			(project "FlexLogicMini_EVB"
 				(path "/483d0913-2604-458a-955b-5458dee34109/5b1eb57d-d000-4da8-a3b9-023ba32e6541"
-					(reference "#PWR0120")
+					(reference "#PWR0122")
 					(unit 1)
 				)
@@
 		(at 178.689 89.662 0)
 		(unit 1)
+		(body_style 1)
 		(exclude_from_sim no)
 		(in_bom yes)
 		(on_board yes)
+		(in_pos_files yes)
 		(dnp no)
-		(property "Reference" "#PWR0115"
+		(property "Reference" "#PWR0121"
 			(at 178.689 93.472 0)
+			(hide yes)
+			(show_name no)
+			(do_not_autoplace no)
 			(effects
 				(font
 					(size 1.27 1.27)
 				)
-				(hide yes)
 			)
 		)
 		(property "Value" "+3.3V_D"
 			(at 178.562 86.106 0)
+			(show_name no)
+			(do_not_autoplace no)
 			(effects
 				(font
@@
 		(property "Footprint" ""
 			(at 178.689 89.662 0)
+			(hide yes)
+			(show_name no)
+			(do_not_autoplace no)
 			(effects
 				(font
 					(size 1.27 1.27)
 				)
-				(hide yes)
 			)
 		)
 		(property "Datasheet" ""
 			(at 178.689 89.662 0)
+			(hide yes)
+			(show_name no)
+			(do_not_autoplace no)
 			(effects
 				(font
 					(size 1.27 1.27)
 				)
-				(hide yes)
 			)
 		)
 		(property "Description" "Power symbol creates a global label with name \"+3.3V\""
 			(at 178.689 89.662 0)
+			(hide yes)
+			(show_name no)
+			(do_not_autoplace no)
 			(effects
 				(font
 					(size 1.27 1.27)
 				)
-				(hide yes)
 			)
 		)
@@
 		)
 		(instances
-			(project "FT2232H_EVB"
+			(project "FlexLogicMini_EVB"
 				(path "/483d0913-2604-458a-955b-5458dee34109/5b1eb57d-d000-4da8-a3b9-023ba32e6541"
-					(reference "#PWR0115")
+					(reference "#PWR0121")
 					(unit 1)
 				)
@@
 		(at 176.403 107.569 0)
 		(unit 1)
+		(body_style 1)
 		(exclude_from_sim no)
 		(in_bom yes)
 		(on_board yes)
+		(in_pos_files yes)
 		(dnp no)
-		(property "Reference" "U12"
+		(property "Reference" "U11"
 			(at 171.958 99.441 0)
+			(show_name no)
+			(do_not_autoplace no)
 			(effects
 				(font
@@
 		(property "Value" "TMUX1574DYYR"
 			(at 158.877 102.108 0)
+			(show_name no)
+			(do_not_autoplace no)
 			(effects
 				(font
@@
 		(property "Footprint" "TMUX1574DYYR:SOT-23-THIN-16_DYY_TEX"
 			(at 176.911 121.539 0)
+			(hide yes)
+			(show_name no)
+			(do_not_autoplace no)
 			(effects
 				(font
@@
 					(italic yes)
 				)
-				(hide yes)
 			)
 		)
 		(property "Datasheet" "TMUX1574DYYR"
 			(at 173.863 117.475 0)
+			(hide yes)
+			(show_name no)
+			(do_not_autoplace no)
 			(effects
 				(font
@@
 					(italic yes)
 				)
-				(hide yes)
 			)
 		)
 		(property "Description" ""
 			(at 196.215 107.569 0)
+			(hide yes)
+			(show_name no)
+			(do_not_autoplace no)
 			(effects
 				(font
 					(size 1.27 1.27)
 				)
-				(hide yes)
 			)
 		)
 		(property "LCSC" "https://www.lcsc.com/product-detail/Analog-Switches-Multiplexers_Texas-Instruments-TMUX1574DYYR_C1855769.html"
 			(at 195.707 125.095 0)
+			(hide yes)
+			(show_name no)
+			(do_not_autoplace no)
 			(effects
 				(font
 					(size 1.27 1.27)
 				)
-				(hide yes)
 			)
 		)
 		(property "JLCPCB" "C1855769"
 			(at 176.403 107.569 0)
+			(hide yes)
+			(show_name no)
+			(do_not_autoplace no)
 			(effects
 				(font
 					(size 1.27 1.27)
 				)
-				(hide yes)
 			)
 		)
 		(property "MANUFACTURER_PART_NUMBER" "TMUX1574DYYR"
 			(at 176.403 107.569 0)
+			(hide yes)
+			(show_name no)
+			(do_not_autoplace no)
 			(effects
 				(font
 					(size 1.27 1.27)
 				)
-				(hide yes)
 			)
 		)
@@
 		)
 		(instances
-			(project "FT2232H_EVB"
+			(project "FlexLogicMini_EVB"
 				(path "/483d0913-2604-458a-955b-5458dee34109/5b1eb57d-d000-4da8-a3b9-023ba32e6541"
-					(reference "U12")
+					(reference "U11")
 					(unit 1)
 				)

Commit message: V2 commit
Parts:
- renumbered C77 to C79
Changed lines of the file:
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@@
 		(in_pos_files yes)
 		(dnp no)
-		(property "Reference" "C77"
+		(property "Reference" "C79"
 			(at 191.008 93.091 0)
 			(show_name no)
@@
 			(project "FlexLogicMini_EVB"
 				(path "/483d0913-2604-458a-955b-5458dee34109/5b1eb57d-d000-4da8-a3b9-023ba32e6541"
-					(reference "C77")
+					(reference "C79")
 					(unit 1)
 				)
@@
 		(in_pos_files yes)
 		(dnp no)
-		(property "Reference" "#PWR0123"
+		(property "Reference" "#PWR0129"
 			(at 186.563 104.521 0)
 			(hide yes)
@@
 			(project "FlexLogicMini_EVB"
 				(path "/483d0913-2604-458a-955b-5458dee34109/5b1eb57d-d000-4da8-a3b9-023ba32e6541"
-					(reference "#PWR0123")
+					(reference "#PWR0129")
 					(unit 1)
 				)
@@
 		(in_pos_files yes)
 		(dnp no)
-		(property "Reference" "#PWR0122"
+		(property "Reference" "#PWR0128"
 			(at 178.689 158.75 0)
 			(hide yes)
@@
 			(project "FlexLogicMini_EVB"
 				(path "/483d0913-2604-458a-955b-5458dee34109/5b1eb57d-d000-4da8-a3b9-023ba32e6541"
-					(reference "#PWR0122")
+					(reference "#PWR0128")
 					(unit 1)
 				)
@@
 		(in_pos_files yes)
 		(dnp no)
-		(property "Reference" "#PWR0121"
+		(property "Reference" "#PWR0127"
 			(at 178.689 93.472 0)
 			(hide yes)
@@
 			(project "FlexLogicMini_EVB"
 				(path "/483d0913-2604-458a-955b-5458dee34109/5b1eb57d-d000-4da8-a3b9-023ba32e6541"
-					(reference "#PWR0121")
+					(reference "#PWR0127")
 					(unit 1)
 				)

Commit message: V3 commit
Parts:
- removed C79: 0.1uF, Capacitor_SMD:C_0201_0603Metric_Pad0.64x0.40mm_HandSolder, symbol Device:C_Small
- added C77: 0.1uF, Capacitor_SMD:C_0402_1005Metric, symbol Device:C_Small
Connections:
- net +3.3V_D: now also C77.1
- net GND: now also C77.2
